File: rp2040-reference-design.kicad_pcb (KiCad board)
At the start: 4 copper layers, 29.5 x 27 mm, 36 parts, among them J1 Conn_02x05_Odd_Even, J2 Conn_01x10_Pin, J3 Conn_01x10_Pin, U1 RP2040, U2 W25Q128JVS, Y1 12mhz ABM8-272-T

Commit message: fix: drc problems
Routing:
- net GND: vias 37 -> 51
Changed lines of the file:
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@@
 			(crossoutdnponfab yes)
 			(subtractmaskfromsilk no)
-			(outputformat 1)
+			(outputformat 4)
 			(mirror no)
-			(drillshape 1)
+			(drillshape 0)
 			(scaleselection 1)
 			(outputdirectory "")
@@
 	)
 	(via
-		(at 132.5 96)
+		(at 132.5 95)
 		(size 0.6)
 		(drill 0.3)
@@
 	)
 	(via
-		(at 129 89)
+		(at 130 89.5)
 		(size 0.6)
 		(drill 0.3)
@@
 	)
 	(via
-		(at 127 87.5)
+		(at 126.5 87.5)
 		(size 0.6)
 		(drill 0.3)
@@
 	)
 	(via
+		(at 133.044652 99.749575)
+		(size 0.6)
+		(drill 0.3)
+		(layers "F.Cu" "B.Cu")
+		(free yes)
+		(net 1)
+	)
+	(via
 		(at 113 96.5)
 		(size 0.6)
@@
 	)
 	(via
-		(at 130 104)
+		(at 129.5 103.5)
+		(size 0.6)
+		(drill 0.3)
+		(layers "F.Cu" "B.Cu")
+		(free yes)
+		(net 1)
+	)
+	(via
+		(at 128 89.5)
 		(size 0.6)
 		(drill 0.3)
@@
 	)
 	(via
+		(at 127 89.5)
+		(size 0.6)
+		(drill 0.3)
+		(layers "F.Cu" "B.Cu")
+		(free yes)
+		(net 1)
+	)
+	(via
 		(at 126.5 95)
 		(size 0.6)
@@
 	)
 	(via
+		(at 117.5 98.5)
+		(size 0.6)
+		(drill 0.3)
+		(layers "F.Cu" "B.Cu")
+		(free yes)
+		(net 1)
+	)
+	(via
+		(at 126 88.5)
+		(size 0.6)
+		(drill 0.3)
+		(layers "F.Cu" "B.Cu")
+		(free yes)
+		(net 1)
+	)
+	(via
 		(at 128 98)
 		(size 0.6)
@@
 	)
 	(via
+		(at 129 89.5)
+		(size 0.6)
+		(drill 0.3)
+		(layers "F.Cu" "B.Cu")
+		(free yes)
+		(net 1)
+	)
+	(via
 		(at 132.5 107)
 		(size 0.6)
@@
 	)
 	(via
-		(at 122.5 107)
+		(at 122.5 105.425)
+		(size 0.6)
+		(drill 0.3)
+		(layers "F.Cu" "B.Cu")
+		(free yes)
+		(net 1)
+	)
+	(via
+		(at 122.5 107.5)
 		(size 0.6)
 		(drill 0.3)
@@
 	)
 	(via
+		(at 129.5 104.5)
+		(size 0.6)
+		(drill 0.3)
+		(layers "F.Cu" "B.Cu")
+		(free yes)
+		(net 1)
+	)
+	(via
 		(at 134 102)
 		(size 0.6)
@@
 	)
 	(via
+		(at 115.5 93.5)
+		(size 0.6)
+		(drill 0.3)
+		(layers "F.Cu" "B.Cu")
+		(free yes)
+		(net 1)
+	)
+	(via
 		(at 125 96.5)
 		(size 0.6)
@@
 	)
 	(via
+		(at 118 89.5)
+		(size 0.6)
+		(drill 0.3)
+		(layers "F.Cu" "B.Cu")
+		(free yes)
+		(net 1)
+	)
+	(via
 		(at 116.5 107)
 		(size 0.6)
@@
 	)
 	(via
+		(at 116 90.5)
+		(size 0.6)
+		(drill 0.3)
+		(layers "F.Cu" "B.Cu")
+		(free yes)
+		(net 1)
+	)
+	(via
+		(at 126.5 86.5)
+		(size 0.6)
+		(drill 0.3)
+		(layers "F.Cu" "B.Cu")
+		(free yes)
+		(net 1)
+	)
+	(via
+		(at 131.5 102)
+		(size 0.6)
+		(drill 0.3)
+		(layers "F.Cu" "B.Cu")
+		(free yes)
+		(net 1)
+	)
+	(via
 		(at 132.5 91)
 		(size 0.6)
@@
 		(net 1)
 	)
+	(via
+		(at 132.5 96.5)
+		(size 0.6)
+		(drill 0.3)
+		(layers "F.Cu" "B.Cu")
+		(free yes)
+		(net 1)
+	)
 	(segment
 		(start 123.15147 102.5)
@@
 	)
 	(segment
+		(start 118.288 106.5)
+		(end 117.474 105.686)
+		(width 0.15)
+		(layer "F.Cu")
+		(net 4)
+	)
+	(segment
 		(start 129 106)
 		(end 129 111.72)
@@
 	)
 	(segment
-		(start 117.474 105.686)
-		(end 117.474 101.532)
+		(start 128.314588 106.5)
+		(end 128.238588 106.424)
 		(width 0.15)
 		(layer "F.Cu")
@@
 	)
 	(segment
-		(start 117.788 106)
-		(end 117.474 105.686)
+		(start 129.43742 100.5)
+		(end 130.023612 100.5)
 		(width 0.15)
 		(layer "F.Cu")
@@
 	)
 	(segment
-		(start 129.43742 100.5)
-		(end 130.023612 100.5)
+		(start 129.28642 100.651)
+		(end 129.43742 100.5)
 		(width 0.15)
 		(layer "F.Cu")
@@
 	)
 	(segment
-		(start 129.28642 100.651)
-		(end 129.43742 100.5)
+		(start 117.474 105.686)
+		(end 117.474 101.532)
 		(width 0.15)
 		(layer "F.Cu")
@@
 	)
 	(segment
+		(start 115.902 99.96)
+		(end 115.05 99.96)
+		(width 0.15)
+		(layer "F.Cu")
+		(net 4)
+	)
+	(segment
+		(start 129 106)
+		(end 128.5 106.5)
+		(width 0.15)
+		(layer "F.Cu")
+		(net 4)
+	)
+	(segment
 		(start 132.5 102.5)
 		(end 129 106)
@@
 	)
 	(segment
-		(start 115.902 99.96)
-		(end 115.05 99.96)
+		(start 128.238588 106.424)
+		(end 127.761412 106.424)
 		(width 0.15)
 		(layer "F.Cu")
@@
 	)
 	(segment
+		(start 127.761412 106.424)
+		(end 127.685412 106.5)
+		(width 0.15)
+		(layer "F.Cu")
+		(net 4)
+	)
+	(segment
 		(start 115.05 98.03)
 		(end 115.02 98)
@@
 	)
 	(segment
-		(start 129 106)
-		(end 117.788 106)
+		(start 127.685412 106.5)
+		(end 118.288 106.5)
+		(width 0.15)
+		(layer "F.Cu")
+		(net 4)
+	)
+	(segment
+		(start 128.5 106.5)
+		(end 128.314588 106.5)
 		(width 0.15)
 		(layer "F.Cu")

Commit message: feat: did stuff
Routing:
- net GPIO19: track 15.9 -> 19.1 mm
- net GND: track 12.1 -> 12.6 mm, vias 51 -> 53
