File: rp2040-reference-design.kicad_pcb (KiCad board)
At the start: 4 copper layers, 29.5 x 27 mm, 36 parts, among them J1 Conn_02x05_Odd_Even, J2 Conn_01x10_Pin, J3 Conn_01x10_Pin, U1 RP2040, U2 W25Q128JVS, Y1 12mhz ABM8-272-T

Commit message: feat: annotated stuff
Parts:
- renumbered J1 to BMDU
Changed lines of the file:
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@@
 	(net 13 "SWDCLK")
 	(net 14 "SWDIO")
-	(net 15 "unconnected-(J1-Pin_8-Pad8)")
-	(net 16 "unconnected-(J1-Pin_6-Pad6)")
+	(net 15 "unconnected-(BMDU1-Pin_8-Pad8)")
+	(net 16 "unconnected-(BMDU1-Pin_6-Pad6)")
 	(net 17 "GPIO8")
 	(net 18 "GPIO7")
@@
 		(descr "surface-mounted straight pin header, 2x05, 1.27mm pitch, double rows")
 		(tags "Surface mounted pin header SMD 2x05 1.27mm double row")
-		(property "Reference" "J1"
+		(property "Reference" "BMDU"
 			(at -0.00718 3.772841 0)
 			(layer "F.SilkS")
@@
 			(size 2.4 0.74)
 			(layers "F.Cu" "F.Mask" "F.Paste")
-			(net 16 "unconnected-(J1-Pin_6-Pad6)")
+			(net 16 "unconnected-(BMDU1-Pin_6-Pad6)")
 			(pinfunction "Pin_6")
 			(pintype "passive+no_connect")
@@
 			(size 2.4 0.74)
 			(layers "F.Cu" "F.Mask" "F.Paste")
-			(net 15 "unconnected-(J1-Pin_8-Pad8)")
+			(net 15 "unconnected-(BMDU1-Pin_8-Pad8)")
 			(pinfunction "Pin_8")
 			(pintype "passive+no_connect")
@@
 	)
 	(segment
-		(start 130.761412 105.924)
-		(end 130.685412 106)
+		(start 122.5 104.5)
+		(end 122.5 101)
 		(width 0.15)
 		(layer "B.Cu")
@@
 	)
 	(segment
-		(start 131.238588 105.924)
-		(end 130.761412 105.924)
+		(start 135.38 106)
+		(end 124 106)
 		(width 0.15)
 		(layer "B.Cu")
@@
 	)
 	(segment
-		(start 131.314588 106)
-		(end 131.238588 105.924)
-		(width 0.15)
-		(layer "B.Cu")
-		(net 28)
-	)
-	(segment
-		(start 130.685412 106)
-		(end 124 106)
-		(width 0.15)
-		(layer "B.Cu")
-		(net 28)
-	)
-	(segment
-		(start 122.5 104.5)
-		(end 122.5 101)
-		(width 0.15)
-		(layer "B.Cu")
-		(net 28)
-	)
-	(segment
-		(start 135.38 106)
-		(end 131.314588 106)
-		(width 0.15)
-		(layer "B.Cu")
-		(net 28)
-	)
-	(segment
 		(start 136 105.38)
 		(end 135.38 106)
@@
 	)
 	(segment
-		(start 130.540023 105.649)
-		(end 130.616024 105.573)
-		(width 0.15)
-		(layer "B.Cu")
-		(net 29)
-	)
-	(segment
-		(start 131.459977 105.649)
-		(end 133.191 105.649)
-		(width 0.15)
-		(layer "B.Cu")
-		(net 29)
-	)
-	(segment
-		(start 130.616024 105.573)
-		(end 131.383976 105.573)
-		(width 0.15)
-		(layer "B.Cu")
-		(net 29)
-	)
-	(segment
-		(start 131.383976 105.573)
-		(end 131.459977 105.649)
+		(start 123.575337 105.078949)
+		(end 124.145388 105.649)
 		(width 0.15)
 		(layer "B.Cu")
@@
 	)
 	(segment
-		(start 124.145388 105.649)
-		(end 130.540023 105.649)
-		(width 0.15)
-		(layer "B.Cu")
-		(net 29)
-	)
-	(segment
 		(start 123.575337 101.075337)
 		(end 123.575337 105.078949)
@@
 	)
 	(segment
-		(start 123.575337 105.078949)
-		(end 124.145388 105.649)
+		(start 124.145388 105.649)
+		(end 133.191 105.649)
 		(width 0.15)
 		(layer "B.Cu")
